File: Pieces/dimmer_led/Dimmer.kicad_sch (KiCad schematic)
At the start: 39 parts, among them J1 Conn_01x02_Female, J2 Conn_01X03, J3 TB_1X6, J4 Conn_01x03_Female, Q1 BTA06-600C, Q2 BTA06-600C, Q3 BTA06-600C, Q5 2N7000, U1 LM78XX, U14 LM324, U3 MOC3020M, U4 MOC3020M, U5 MOC3020M, U7 PC817

Commit message: terminado dimmer
Parts:
- removed J3: TB_1X6, symbol Dimmer-rescue:TB_1X6-MacroLib
- added J3, J5, J6: TB_1X2, EESTN5:BORNERA2, symbol EESTN5:TB_1X2
- C1, C2, C20, C21, C22, C23: footprint EESTN5:C_0805 -> EESTN5:C_1206
- D6: footprint (none) -> EESTN5:Diode_Bridge_Round_D8.9mm
- J1: footprint (none) -> EESTN5:Pin_strip_2
- J2: footprint (none) -> EESTN5:Pin_Strip_3
- J4: footprint Connector:FanPinHeader_1x03_P2.54mm_Vertical -> MacroLib:FanPinHeader_1x03_P2.54mm_Vertical
- Q5: footprint (none) -> EESTN5:to92
- R20, R21, R22, R24, R25, R26, R28, R29, R30, R31, R32, R33, R34, R35, R36, R37, R38, R46: footprint (none) -> EESTN5:R_1206
- U1: footprint (none) -> MacroLib:TO-220-3_Vertical
- U14: footprint (none) -> MacroLib:DIP-14
- U3, U4, U5: footprint (none) -> MacroLib:DIP-6
- U7: footprint Housings_DIP:DIP-4_W7.62mm -> MacroLib:DIP-4
Connections:
- net Earth: now also J3.2, J5.2, J6.2
- net at Q1.2 (A2), R24.2: now also J3.1
- net at Q2.2 (A2), R25.1: now also J5.1
- net at Q3.2 (A2), R26.1: now also J6.1

Commit message: lista de componentes
Parts:
- renumbered C20 to C3, C21 to C4, C23 to C5, C22 to C6, D6 to D1, J3 to J2, J2 to J3, J5 to J4, J6 to J5, J4 to J6, Q5 to Q1, Q1 to Q2, Q2 to Q3, Q3 to Q4, R32 to R1, R46 to R10, R20 to R11, R24 to R12, R21 to R13, R25 to R14, R35 to R15, R22 to R16, R26 to R17, R37 to R18, R29 to R2, R28 to R3, R30 to R4, R31 to R5, R33 to R6, R34 to R7, R38 to R8, R36 to R9, U7 to U2, U14 to U3, U3 to U4, U4 to U5, U5 to U6

Commit message: dimmer actualizado
Parts:
- C1, C4, C5, C6: footprint EESTN5:C_1206 -> EESTN5:CAP_0.1
- C2, C3: footprint EESTN5:C_1206 -> EESTN5:C_0805
- R11, R13, R16: footprint EESTN5:R_1206 -> EESTN5:R_0805
- R2, R4, R6: footprint EESTN5:R_1206 -> EESTN5:RES0.2
- R3: footprint EESTN5:R_1206 -> EESTN5:RES0.3
Changed lines of the file:
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@@
     (property "Reference" "R3" (id 0) (at 74.93 54.61 90))
     (property "Value" "33k" (id 1) (at 80.01 54.61 90))
-    (property "Footprint" "EESTN5:R_1206" (id 2) (at 77.47 57.15 0)
+    (property "Footprint" "EESTN5:RES0.3" (id 2) (at 77.47 57.15 0)
       (effects (font (size 1.524 1.524)) hide)
     )
@@
       (effects (font (size 1.27 1.27)) (justify left))
     )
-    (property "Footprint" "EESTN5:R_1206" (id 2) (at 100.33 52.07 0)
+    (property "Footprint" "EESTN5:RES0.2" (id 2) (at 100.33 52.07 0)
       (effects (font (size 1.524 1.524)) hide)
     )
@@
     (property "Reference" "R4" (id 0) (at 107.95 52.451 90))
     (property "Value" "1k" (id 1) (at 107.95 54.7624 90))
-    (property "Footprint" "EESTN5:R_1206" (id 2) (at 107.95 57.15 0)
+    (property "Footprint" "EESTN5:RES0.2" (id 2) (at 107.95 57.15 0)
       (effects (font (size 1.524 1.524)) hide)
     )
@@
       (effects (font (size 1.27 1.27)) (justify left))
     )
-    (property "Footprint" "EESTN5:R_1206" (id 2) (at 120.65 66.04 0)
+    (property "Footprint" "EESTN5:RES0.2" (id 2) (at 120.65 66.04 0)
       (effects (font (size 1.524 1.524)) hide)
     )
@@
       (effects (font (size 1.016 1.016)) (justify left))
     )
-    (property "Footprint" "EESTN5:C_1206" (id 2) (at 135.5852 66.04 0)
+    (property "Footprint" "EESTN5:C_0805" (id 2) (at 135.5852 66.04 0)
       (effects (font (size 0.762 0.762)) hide)
     )
@@
       (effects (font (size 1.016 1.016)) (justify left))
     )
-    (property "Footprint" "EESTN5:C_1206" (id 2) (at 178.7652 88.9 0)
+    (property "Footprint" "EESTN5:CAP_0.1" (id 2) (at 178.7652 88.9 0)
       (effects (font (size 0.762 0.762)) hide)
     )
@@
       (effects (font (size 1.016 1.016)) (justify left))
     )
-    (property "Footprint" "EESTN5:C_1206" (id 2) (at 235.9152 88.9 0)
+    (property "Footprint" "EESTN5:CAP_0.1" (id 2) (at 235.9152 88.9 0)
       (effects (font (size 0.762 0.762)) hide)
     )
@@
     (property "Reference" "R16" (id 0) (at 43.18 122.301 90))
     (property "Value" "220" (id 1) (at 43.18 124.6124 90))
-    (property "Footprint" "EESTN5:R_1206" (id 2) (at 43.18 127 0)
+    (property "Footprint" "EESTN5:R_0805" (id 2) (at 43.18 127 0)
       (effects (font (size 1.524 1.524)) hide)
     )
@@
     (property "Reference" "R13" (id 0) (at 43.18 112.141 90))
     (property "Value" "220" (id 1) (at 43.18 114.4524 90))
-    (property "Footprint" "EESTN5:R_1206" (id 2) (at 43.18 116.84 0)
+    (property "Footprint" "EESTN5:R_0805" (id 2) (at 43.18 116.84 0)
       (effects (font (size 1.524 1.524)) hide)
     )
@@
     (property "Reference" "R11" (id 0) (at 43.18 101.981 90))
     (property "Value" "220" (id 1) (at 43.18 104.2924 90))
-    (property "Footprint" "EESTN5:R_1206" (id 2) (at 43.18 106.68 0)
+    (property "Footprint" "EESTN5:R_0805" (id 2) (at 43.18 106.68 0)
       (effects (font (size 1.524 1.524)) hide)
     )
@@
       (effects (font (size 1.016 1.016)) (justify left))
     )
-    (property "Footprint" "EESTN5:C_1206" (id 2) (at 178.7652 137.16 0)
+    (property "Footprint" "EESTN5:CAP_0.1" (id 2) (at 178.7652 137.16 0)
       (effects (font (size 0.762 0.762)) hide)
     )
@@
       (effects (font (size 1.016 1.016)) (justify left))
     )
-    (property "Footprint" "EESTN5:C_1206" (id 2) (at 209.2452 41.91 0)
+    (property "Footprint" "EESTN5:CAP_0.1" (id 2) (at 209.2452 41.91 0)
       (effects (font (size 0.762 0.762)) hide)
     )
@@
       (effects (font (size 1.016 1.016)) (justify left))
     )
-    (property "Footprint" "EESTN5:C_1206" (id 2) (at 237.1852 41.91 0)
+    (property "Footprint" "EESTN5:C_0805" (id 2) (at 237.1852 41.91 0)
       (effects (font (size 0.762 0.762)) hide)
     )
@@
     )
     (path "/00000000-0000-0000-0000-000062bcbd60"
-      (reference "C1") (unit 1) (value "220nf") (footprint "EESTN5:C_1206")
+      (reference "C1") (unit 1) (value "220nf") (footprint "EESTN5:CAP_0.1")
     )
     (path "/00000000-0000-0000-0000-000062bcc2e0"
-      (reference "C2") (unit 1) (value "100nf") (footprint "EESTN5:C_1206")
+      (reference "C2") (unit 1) (value "100nf") (footprint "EESTN5:C_0805")
     )
     (path "/00000000-0000-0000-0000-0000628a61c0"
-      (reference "C3") (unit 1) (value "100nf") (footprint "EESTN5:C_1206")
+      (reference "C3") (unit 1) (value "100nf") (footprint "EESTN5:C_0805")
     )
     (path "/00000000-0000-0000-0000-0000628d8880"
-      (reference "C4") (unit 1) (value "1uf") (footprint "EESTN5:C_1206")
+      (reference "C4") (unit 1) (value "1uf") (footprint "EESTN5:CAP_0.1")
     )
     (path "/00000000-0000-0000-0000-0000629e713f"
-      (reference "C5") (unit 1) (value "1uf") (footprint "EESTN5:C_1206")
+      (reference "C5") (unit 1) (value "1uf") (footprint "EESTN5:CAP_0.1")
     )
     (path "/00000000-0000-0000-0000-000062a801ce"
-      (reference "C6") (unit 1) (value "1uf") (footprint "EESTN5:C_1206")
+      (reference "C6") (unit 1) (value "1uf") (footprint "EESTN5:CAP_0.1")
     )
     (path "/00000000-0000-0000-0000-00006289c3d7"
@@
     )
     (path "/00000000-0000-0000-0000-00006289ff43"
-      (reference "R2") (unit 1) (value "1k") (footprint "EESTN5:R_1206")
+      (reference "R2") (unit 1) (value "1k") (footprint "EESTN5:RES0.2")
     )
     (path "/00000000-0000-0000-0000-00006289e570"
-      (reference "R3") (unit 1) (value "33k") (footprint "EESTN5:R_1206")
+      (reference "R3") (unit 1) (value "33k") (footprint "EESTN5:RES0.3")
     )
     (path "/00000000-0000-0000-0000-0000628a32af"
-      (reference "R4") (unit 1) (value "1k") (footprint "EESTN5:R_1206")
+      (reference "R4") (unit 1) (value "1k") (footprint "EESTN5:RES0.2")
     )
     (path "/00000000-0000-0000-0000-0000628a4302"
@@
     )
     (path "/00000000-0000-0000-0000-0000628a5aca"
-      (reference "R6") (unit 1) (value "1k") (footprint "EESTN5:R_1206")
+      (reference "R6") (unit 1) (value "1k") (footprint "EESTN5:RES0.2")
     )
     (path "/00000000-0000-0000-0000-0000628cf870"
@@
     )
     (path "/00000000-0000-0000-0000-000062a40cbd"
-      (reference "R11") (unit 1) (value "220") (footprint "EESTN5:R_1206")
+      (reference "R11") (unit 1) (value "220") (footprint "EESTN5:R_0805")
     )
     (path "/00000000-0000-0000-0000-0000629ee71a"
@@
     )
     (path "/00000000-0000-0000-0000-000062a406bc"
-      (reference "R13") (unit 1) (value "220") (footprint "EESTN5:R_1206")
+      (reference "R13") (unit 1) (value "220") (footprint "EESTN5:R_0805")
     )
     (path "/00000000-0000-0000-0000-0000629eecfc"
@@
     )
     (path "/00000000-0000-0000-0000-000062a3ff6b"
-      (reference "R16") (unit 1) (value "220") (footprint "EESTN5:R_1206")
+      (reference "R16") (unit 1) (value "220") (footprint "EESTN5:R_0805")
     )
     (path "/00000000-0000-0000-0000-0000629fa156"
